Commit message: rename

File: echo_bot_description/urdf/EchoBot_wheel.transmission.xacro (robot description, xacro)
@@ -1,33 +1,33 @@
 <?xml version="1.0"?>
 <robot name="EchoBot" xmlns:xacro="http://ros.org/wiki/xacro">
-  <xacro:macro name="joint_position_trans_v0" params="name">
-    <transmission name="${name}_trans">
+  <xacro:macro name="joint_position_trans_v0" params="prefix">
+    <transmission name="${prefix}_trans">
       <type>transmission_interface/SimpleTransmission</type>
-      <joint name="${name}">
+      <joint name="${prefix}">
         <hardwareInterface>PositionJointInterface</hardwareInterface>
       </joint>
-      <actuator name="${name}_motor">
+      <actuator name="${prefix}_motor">
         <hardwareInterface>PositionJointInterface</hardwareInterface>
       </actuator>
     </transmission>
   </xacro:macro>
-  <xacro:macro name="joint_velocity_trans_v0" params="name">
-    <transmission name="${name}_trans">
+  <xacro:macro name="joint_velocity_trans_v0" params="prefix">
+    <transmission name="${prefix}_trans">
       <type>transmission_interface/SimpleTransmission</type>
-      <joint name="${name}">
+      <joint name="${prefix}">
         <hardwareInterface>VelocityJointInterface</hardwareInterface>
       </joint>
-      <actuator name="${name}_motor">
+      <actuator name="${prefix}_motor">
         <hardwareInterface>VelocityJointInterface</hardwareInterface>
       </actuator>
     </transmission>
   </xacro:macro>
-  <xacro:macro name="joint_effort_trans_v0" params="name">
-    <transmission name="${name}_trans">
+  <xacro:macro name="joint_effort_trans_v0" params="prefix">
+    <transmission name="${prefix}_trans">
       <type>transmission_interface/SimpleTransmission</type>
-      <joint name="${name}">
+      <joint name="${prefix}">
         <hardwareInterface>EffortJointInterface</hardwareInterface>
       </joint>
-      <actuator name="${name}_motor">
+      <actuator name="${prefix}_motor">
         <hardwareInterface>EffortJointInterface</hardwareInterface>
       </actuator>
