Commit message: fix R to L

File: echo_bot_description/robot/echo_bot.urdf.xacro (robot description, xacro)
@@ -1,8 +1,26 @@
 <?xml version="1.0"?>
 <robot name="echo_bot" xmlns:xacro="http://ros.org/wiki/xacro">
+  <xacro:include filename="$(find echo_bot_description)/urdf/common.xacro"/>
+  <xacro:include filename="$(find echo_bot_description)/urdf/base/echo_bot_base.urdf.xacro"/>
+  <xacro:include filename="$(find echo_bot_description)/urdf/leg/echo_bot_left_leg.urdf.xacro"/>
+  <xacro:include filename="$(find echo_bot_description)/urdf/wheel/echo_bot_wheel.urdf.xacro"/>
+  <!-- <xacro:include filename="$(find echo_bot_description)/urdf/SENSOR.urdf.xacro"/> -->
   <!-- == echo_bot base == -->
-  <xacro:include filename="$(find echo_bot_description)/urdf/echo_bot_base.urdf.xacro"/>
+  <link name="base_footprint"/>
+  <xacro:base_v0 parent="base_footprint">
+  <origin xyz="0 0 0.090"/>
+  </xacro:base_v0>
+  <!-- == left_leg == -->
+  <xacro:left_leg_v0 parent="base_link">
+    <origin xyz="0.0 0.0475 0.0" rpy="0.0 ${M_PI*160/180} 0.0"/>
+  </xacro:left_leg_v0>
+  <xacro:wheel_v0 prefix="left" parent="lower_leg_L">
+    <origin xyz="0.1 0.0305 0.0" rpy="${-M_PI/2} 0.0 0.0"/>
+    <axis xyz="0 0 1"/>
+  </xacro:wheel_v0>
+  <xacro:joint_velocity_trans_v0 prefix="left"/>
+  <!-- == right_leg == -->
+  <!-- <xacro:include filename="$(find echo_bot_description)/urdf/leg/echo_bot_right_leg.urdf.xacro"/> -->
   <!-- == Sensor == -->
-  <!-- <xacro:include filename="$(find echo_bot_description)/urdf/SENSOR.urdf.xacro"/> -->
   <!-- == Gazebo == -->
   <gazebo>
@@ -14,6 +32,6 @@
   <xacro:base_gazebo_v0/>
   <!-- Wheel -->
-  <xacro:wheel_gazebo_v0 prefix="right"/>
   <xacro:wheel_gazebo_v0 prefix="left"/>
+  <!-- <xacro:wheel_gazebo_v0 prefix="right"/> -->
   <!-- <xacro:wheel_gazebo_control_v0 rate="25"/> -->
 </robot>

File: echo_bot_description/robot/test.urdf (robot description, URDF)
Before this commit: robot echo_bot, 6 links, 5 joints
Links:
- removed link Body
- removed link lower_leg_R
- removed link upper_leg_R
- removed link upper_side_leg_R
- added link base_link, mass 1e-06; collision mesh filename=package://echo_bot_description/meshes/STL/body.stl; visual mesh filename=package://echo_bot_description/meshes/STL/body.stl
- added link lower_leg_L, mass 13.25; collision mesh filename=package://echo_bot_description/meshes/STL/lower_leg.stl; visual mesh filename=package://echo_bot_description/meshes/STL/lower_leg.stl
- added link upper_leg_L, mass 13.25; collision mesh filename=package://echo_bot_description/meshes/STL/upper_leg.stl; visual mesh filename=package://echo_bot_description/meshes/STL/upper_leg.stl
- added link upper_side_leg_L, mass 13.25; collision mesh filename=package://echo_bot_description/meshes/STL/upper_side_leg.stl; visual mesh filename=package://echo_bot_description/meshes/STL/upper_side_leg.stl
Joints:
- removed joint base_footprint_to_Body
- removed joint lower_leg_R
- removed joint upper_leg_R
- removed joint upper_side_leg_R
- added joint base_link_joint: type fixed, parent base_footprint, child base_link, origin xyz=0 0 0.090
- added joint lower_leg_L: type revolute, parent upper_leg_L, child lower_leg_L, origin xyz=0.1 0.0 0.0 rpy=0.0 -2.52147723971 0.0, axis 0 1 0, limit lower=0.0 upper=1.16465824189 effort=0 velocity=0, mimic joint=upper_leg_L multiplier=-2.186 offset=-0.02025
- added joint upper_leg_L: type revolute, parent base_link, child upper_leg_L, origin xyz=0.0 0.0475 0.0 rpy=0.0 2.79252688 0.0, axis 0 1 0, limit lower=0.0 upper=-0.52359879 effort=0 velocity=0
- added joint upper_side_leg_L: type revolute, parent lower_leg_L, child upper_side_leg_L, origin xyz=-0.025 0.0 0.0 rpy=0.0 -0.94631754646 0.0, axis 0 1 0, limit lower=0.0 upper=-1.12975165589 effort=0 velocity=0, mimic joint=upper_leg_L multiplier=2.123937 offset=0.003625
- joint wheel_left: parent lower_leg_R -> lower_leg_L

File: echo_bot_description/urdf/leg/echo_bot_left_leg.urdf.xacro (robot description, xacro)
@@ -5,6 +5,7 @@
     <color rgba="0.3 0.3 0.3 1"/>
   </material>
+  <xacro:macro name="left_leg_v0" params="parent *joint_origin">
   <!-- Link -->
-  <link name="upper_leg_R">
+  <link name="upper_leg_L">
     <visual>
       <origin rpy="0 0 0"/>
@@ -26,5 +27,5 @@
     </inertial>
   </link>
-  <link name="lower_leg_R">
+  <link name="lower_leg_L">
     <visual>
       <origin rpy="0 0 0"/>
@@ -46,5 +47,5 @@
     </inertial>
   </link>
-  <link name="upper_side_leg_R">
+  <link name="upper_side_leg_L">
     <visual>
       <origin rpy="0 0 0"/>
@@ -67,34 +68,27 @@
   </link>
   <!-- Joint -->
-  <joint name="upper_leg_R" type="revolute">
-    <origin xyz="0.0 0.0475 0.0" rpy="0.0 ${M_PI*160/180} 0.0" />
-    <parent link="Body" />
-    <child link="upper_leg_R" />
+  <joint name="upper_leg_L" type="revolute">
+    <insert_block name="joint_origin"/>
+    <parent link="${parent}" />
+    <child link="upper_leg_L" />
     <axis xyz="0 1 0"/>
     <limit lower="0.0" upper="${-M_PI*30/180}" effort="0" velocity="0"/>
   </joint>
-  <!-- <xacro:joint_velocity_trans_v0 name="upper_leg_R"/> -->
-  <joint name="lower_leg_R" type="revolute">
+  <joint name="lower_leg_L" type="revolute">
     <origin xyz="0.1 0.0 0.0" rpy="0.0 ${-M_PI*144.47/180} 0.0" />
-    <parent link="upper_leg_R" />
-    <child link="lower_leg_R" />
+    <parent link="upper_leg_L" />
+    <child link="lower_leg_L" />
     <axis xyz="0 1 0"/>
     <limit lower="0.0" upper="${M_PI*66.73/180}" effort="0" velocity="0"/>
-    <mimic joint="upper_leg_R" multiplier="-2.186" offset="-0.02025"/>
+    <mimic joint="upper_leg_L" multiplier="-2.186" offset="-0.02025"/>
   </joint>
-  <joint name="upper_side_leg_R" type="revolute">
+  <joint name="upper_side_leg_L" type="revolute">
     <origin xyz="-0.025 0.0 0.0" rpy="0.0 ${-M_PI*54.22/180} 0.0" />
-    <parent link="lower_leg_R" />
-    <child link="upper_side_leg_R" />
+    <parent link="lower_leg_L" />
+    <child link="upper_side_leg_L" />
     <axis xyz="0 1 0"/>
     <limit lower="0.0" upper="${-M_PI*64.73/180}" effort="0" velocity="0"/>
-    <mimic joint="upper_leg_R" multiplier="2.123937" offset="0.003625"/>
+    <mimic joint="upper_leg_L" multiplier="2.123937" offset="0.003625"/>
   </joint>
-  <xacro:include filename="$(find echo_bot_description)/urdf/wheel/echo_bot_wheel.urdf.xacro"/>
-  <xacro:wheel_v0 prefix="left" parent="lower_leg_R">
-    <origin xyz="0.1 0.0305 0.0" rpy="${-M_PI/2} 0.0 0.0"/>
-    <axis xyz="0 0 1"/>
-  </xacro:wheel_v0>
-  <!-- Transmission -->
-  <xacro:wheel_trans_v0 prefix="right"/>
+  </xacro:macro>
 </robot>
