Commit message: edit something

File: echo_bot_description/urdf/leg/echo_bot_left_leg.gazebo.xacro (robot description, xacro)
@@ -2,15 +2,15 @@
 <robot name="echo_bot" xmlns:xacro="http://ros.org/wiki/xacro">
   <xacro:macro name="left_leg_gazebo_v0">
-    <gazebo reference="upper_leg_L">
+    <gazebo reference="upper_leg_left">
       <selfCollide>true</selfCollide>
       <mu1 value="0.8" />
       <mu2 value="0.8" />
     </gazebo>
-    <gazebo reference="lower_leg_L">
+    <gazebo reference="lower_leg_left">
       <selfCollide>true</selfCollide>
       <mu1 value="0.8" />
       <mu2 value="0.8" />
     </gazebo>
-    <gazebo reference="upper_side_leg_L">
+    <gazebo reference="upper_side_leg_left">
       <selfCollide>true</selfCollide>
       <mu1 value="0.8" />

File: echo_bot_description/urdf/wheel/echo_bot_wheel.gazebo.xacro (robot description, xacro)
@@ -2,5 +2,5 @@
 <robot xmlns:xacro="http://ros.org/wiki/xacro">
   <xacro:macro name="wheel_gazebo_v0" params="prefix">
-    <gazebo reference="${prefix}_wheel_link">
+    <gazebo reference="wheel_${prefix}_link">
       <selfCollide>true</selfCollide>
       <mu1 value="0.8" />

File: echo_bot_description/urdf/wheel/echo_bot_wheel.transmission.xacro (robot description, xacro)
@@ -1,34 +1,13 @@
 <?xml version="1.0"?>
-<robot name="echo_bot" xmlns:xacro="http://ros.org/wiki/xacro">
-  <xacro:macro name="joint_position_trans_v0" params="prefix">
-    <transmission name="${prefix}_trans">
+<robot xmlns:xacro="http://ros.org/wiki/xacro">
+  <xacro:macro name="wheel_trans_v0" params="prefix">
+    <transmission name="wheel_${prefix}_trans">
       <type>transmission_interface/SimpleTransmission</type>
-      <joint name="${prefix}">
-        <hardwareInterface>PositionJointInterface</hardwareInterface>
+      <joint name="wheel_${prefix}_joint">
+        <hardwareInterface>hardware_interface/VelocityJointInterface</hardwareInterface>
       </joint>
-      <actuator name="${prefix}_motor">
-        <hardwareInterface>PositionJointInterface</hardwareInterface>
-      </actuator>
-    </transmission>
-  </xacro:macro>
-  <xacro:macro name="joint_velocity_trans_v0" params="prefix">
-    <transmission name="${prefix}_trans">
-      <type>transmission_interface/SimpleTransmission</type>
-      <joint name="${prefix}">
-        <hardwareInterface>VelocityJointInterface</hardwareInterface>
-      </joint>
-      <actuator name="${prefix}_motor">
-        <hardwareInterface>VelocityJointInterface</hardwareInterface>
-      </actuator>
-    </transmission>
-  </xacro:macro>
-  <xacro:macro name="joint_effort_trans_v0" params="prefix">
-    <transmission name="${prefix}_trans">
-      <type>transmission_interface/SimpleTransmission</type>
-      <joint name="${prefix}">
-        <hardwareInterface>EffortJointInterface</hardwareInterface>
-      </joint>
-      <actuator name="${prefix}_motor">
-        <hardwareInterface>EffortJointInterface</hardwareInterface>
+      <actuator name="wheel_${prefix}_motor">
+        <hardwareInterface>hardware_interface/VelocityJointInterface</hardwareInterface>
+        <mechanicalReduction>30</mechanicalReduction>
       </actuator>
     </transmission>
