Commit message: change effort and velocity params

File: echo_bot_description/urdf/leg/echo_bot_leg.urdf.xacro (robot description, xacro)
@@ -81,5 +81,5 @@
       <child link="upper_leg_${prefix}" />
       <axis xyz="0 1 0"/>
-      <limit lower="0.0" upper="${-M_PI*30/180}" effort="1.0" velocity="10.0"/>
+      <limit lower="0.0" upper="${-M_PI*30/180}" effort="30" velocity="${M_PI}"/>
     </joint>
     <xacro:leg_position_trans_v0 joint="upper_leg_${prefix}_joint"/>
@@ -89,5 +89,5 @@
       <child link="lower_leg_${prefix}" />
       <axis xyz="0 1 0"/>
-      <limit lower="0.0" upper="${M_PI*66.73/180}" effort="1.0" velocity="10.0"/>
+      <limit lower="0.0" upper="${M_PI*66.73/180}" effort="30" velocity="${M_PI}"/>
       <!-- <mimic joint="upper_leg_${prefix}_joint" multiplier="-2.186" offset="-0.02025"/> -->
     </joint>
@@ -98,5 +98,5 @@
       <child link="upper_side_leg_${prefix}" />
       <axis xyz="0 1 0"/>
-      <limit lower="0.0" upper="${-M_PI*64.73/180}" effort="1.0" velocity="10.0"/>
+      <limit lower="0.0" upper="${-M_PI*64.73/180}" effort="30" velocity="${M_PI}"/>
       <!-- <mimic joint="upper_leg_${prefix}_joint" multiplier="2.123937" offset="0.003625"/> -->
     </joint>

Commit message: revoluteだとposition_controlできなかった -> continuousにした

File: echo_bot_description/urdf/leg/echo_bot_leg.urdf.xacro (robot description, xacro)
@@ -81,25 +81,27 @@
       <child link="upper_leg_${prefix}" />
       <axis xyz="0 1 0"/>
-      <limit lower="0.0" upper="${-M_PI*30/180}" effort="30" velocity="${M_PI}"/>
+      <limit lower="0.0" upper="${-M_PI*30/180}" effort="5" velocity="${M_PI}"/>
     </joint>
-    <xacro:leg_position_trans_v0 joint="upper_leg_${prefix}_joint"/>
-    <joint name="lower_leg_${prefix}" type="revolute">
+    <!-- <xacro:leg_position_trans_v0 joint="upper_leg_${prefix}_joint"/> -->
+    <xacro:leg_effort_trans_v0 joint="upper_leg_${prefix}_joint"/>
+    <joint name="lower_leg_${prefix}_joint" type="continuous">
       <origin xyz="0.1 0.0 0.0" rpy="0.0 ${-M_PI*144.47/180} 0.0" />
       <parent link="upper_leg_${prefix}" />
       <child link="lower_leg_${prefix}" />
       <axis xyz="0 1 0"/>
-      <limit lower="0.0" upper="${M_PI*66.73/180}" effort="30" velocity="${M_PI}"/>
+      <!-- <limit lower="0.0" upper="${M_PI*66.73/180}" effort="5" velocity="${M_PI}"/> -->
       <!-- <mimic joint="upper_leg_${prefix}_joint" multiplier="-2.186" offset="-0.02025"/> -->
     </joint>
-    <xacro:leg_position_trans_v0 joint="lower_leg_${prefix}"/>
-    <joint name="upper_side_leg_${prefix}" type="revolute">
+    <xacro:leg_position_trans_v0 joint="lower_leg_${prefix}_joint"/>
+    <joint name="upper_side_leg_${prefix}_joint" type="continuous">
       <origin xyz="-0.025 0.0 0.0" rpy="0.0 ${-M_PI*54.22/180} 0.0" />
       <parent link="lower_leg_${prefix}" />
       <child link="upper_side_leg_${prefix}" />
       <axis xyz="0 1 0"/>
-      <limit lower="0.0" upper="${-M_PI*64.73/180}" effort="30" velocity="${M_PI}"/>
+      <!-- <limit lower="0.0" upper="${-M_PI*64.73/180}" effort="5" velocity="${M_PI}"/>
+      <dynamics damping="5" friction="0.1"/> -->
       <!-- <mimic joint="upper_leg_${prefix}_joint" multiplier="2.123937" offset="0.003625"/> -->
     </joint>
-    <xacro:leg_position_trans_v0 joint="upper_side_leg_${prefix}"/>
+    <xacro:leg_position_trans_v0 joint="upper_side_leg_${prefix}_joint"/>
   </xacro:macro>
 </robot>
