Commit message: change model STL to DAE

File: echo_bot_description/urdf/base/echo_bot_base.urdf.xacro (robot description, xacro)
@@ -1,4 +1,4 @@
 <?xml version="1.0"?>
-<robot name="echo_bot" xmlns:xacro="http://ros.org/wiki/xacro">
+<robot xmlns:xacro="http://ros.org/wiki/xacro">
   <!-- == Material == -->
   <material name="base_color">
@@ -18,5 +18,5 @@
         <origin rpy="0 0 0"/>
         <geometry>
-          <mesh filename="package://echo_bot_description/meshes/STL/body.stl"/>
+          <mesh filename="package://echo_bot_description/meshes/DAE/body.dae"/>
         </geometry>
       </collision>

Commit message: Fix base_link mass value because too little mass becomes 0 due to rounding error

File: echo_bot_description/urdf/base/echo_bot_base.urdf.xacro (robot description, xacro)
@@ -22,5 +22,5 @@
       </collision>
       <inertial>
-        <mass value="1e-06" />
+        <mass value="1e-05" />
         <origin xyz="0 0 0" rpy="0 0 0" />
         <inertia ixx="1.0" ixy="0.0" ixz="0.0" iyy="1.0" iyz="0.0" izz="1.0" />

Commit message: fix model parameter

File: echo_bot_description/urdf/base/echo_bot_base.urdf.xacro (robot description, xacro)
@@ -12,5 +12,5 @@
         <material name="base_color"/>
         <geometry>
-          <mesh filename="package://echo_bot_description/meshes/STL/body.stl"/>
+          <mesh filename="package://echo_bot_description/meshes/DAE/body.dae"/>
         </geometry>
       </visual>
@@ -18,5 +18,5 @@
         <origin rpy="0 0 0"/>
         <geometry>
-          <mesh filename="package://echo_bot_description/meshes/DAE/body.dae"/>
+          <mesh filename="package://echo_bot_description/meshes/STL/body.stl"/>
         </geometry>
       </collision>

File: echo_bot_description/urdf/leg/echo_bot_leg.urdf.xacro (robot description, xacro)
@@ -14,5 +14,5 @@
         <material name="leg_color_0"/>
         <geometry>
-          <mesh filename="package://echo_bot_description/meshes/STL/upper_leg.stl"/>
+          <mesh filename="package://echo_bot_description/meshes/DAE/upper_leg.dae"/>
         </geometry>
       </visual>
@@ -20,5 +20,5 @@
         <origin rpy="0 0 0"/>
         <geometry>
-          <mesh filename="package://echo_bot_description/meshes/DAE/upper_leg.dae"/>
+          <mesh filename="package://echo_bot_description/meshes/STL/upper_leg.stl"/>
         </geometry>
       </collision>
@@ -36,5 +36,5 @@
         <material name="leg_color_0"/>
         <geometry>
-          <mesh filename="package://echo_bot_description/meshes/STL/lower_leg_${prefix}.stl"/>
+          <mesh filename="package://echo_bot_description/meshes/DAE/lower_leg_${prefix}.dae"/>
         </geometry>
       </visual>
@@ -42,5 +42,5 @@
         <origin rpy="0 0 0"/>
         <geometry>
-          <mesh filename="package://echo_bot_description/meshes/DAE/lower_leg_${prefix}.dae"/>
+          <mesh filename="package://echo_bot_description/meshes/STL/lower_leg_${prefix}.stl"/>
         </geometry>
       </collision>
@@ -58,5 +58,5 @@
         <material name="leg_color_0"/>
         <geometry>
-          <mesh filename="package://echo_bot_description/meshes/STL/upper_side_leg.stl"/>
+          <mesh filename="package://echo_bot_description/meshes/DAE/upper_side_leg.dae"/>
         </geometry>
       </visual>
@@ -64,5 +64,5 @@
         <origin rpy="0 0 0"/>
         <geometry>
-          <mesh filename="package://echo_bot_description/meshes/DAE/upper_side_leg.dae"/>
+          <mesh filename="package://echo_bot_description/meshes/STL/upper_side_leg.stl"/>
         </geometry>
       </collision>

File: echo_bot_description/urdf/wheel/echo_bot_wheel.urdf.xacro (robot description, xacro)
@@ -13,5 +13,5 @@
         <material name="wheel_color"/>
         <geometry>
-          <mesh filename="package://echo_bot_description/meshes/STL/tyre.stl"/>
+          <mesh filename="package://echo_bot_description/meshes/DAE/tyre.dae"/>
         </geometry>
       </visual>
@@ -19,5 +19,5 @@
         <origin rpy="0 0 0"/>
         <geometry>
-          <mesh filename="package://echo_bot_description/meshes/DAE/tyre.dae"/>
+          <mesh filename="package://echo_bot_description/meshes/STL/tyre.stl"/>
         </geometry>
       </collision>
