Commit message: cmd_velの設定した→指令値送ったけどなんか動かん

File: echo_bot_description/robots/test.urdf (robot description, URDF)
Before this commit: robot echo_bot, 12 links, 11 joints
Links:
- removed link side_leg_left
- removed link side_leg_right
- removed link world
- added link base_footprint
- link base_link: geometry collision mesh filename=package://echo_bot_description/meshes/STL/body.stl; visual mesh filename=package://echo_bot_description/meshes/DAE/body.dae
- link lower_leg_left: geometry collision mesh filename=package://echo_bot_description/meshes/STL/lower_leg_left.stl; visual mesh filename=package://echo_bot_description/meshes/DAE/lower_leg_left.dae
- link lower_leg_right: geometry collision mesh filename=package://echo_bot_description/meshes/STL/lower_leg_right.s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; visual mesh filename=package://echo_bot_description/meshes/DAE/lower_leg_right.d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
- link upper_leg_left: geometry collision mesh filename=package://echo_bot_description/meshes/STL/upper_leg.stl; visual mesh filename=package://echo_bot_description/meshes/DAE/upper_leg.dae
- link upper_leg_right: geometry collision mesh filename=package://echo_bot_description/meshes/STL/upper_leg.stl; visual mesh filename=package://echo_bot_description/meshes/DAE/upper_leg.dae
- link upper_side_leg_left: geometry collision mesh filename=package://echo_bot_description/meshes/STL/upper_side_leg.stl; visual mesh filename=package://echo_bot_description/meshes/DAE/upper_side_leg.dae
- link upper_side_leg_right: geometry collision mesh filename=package://echo_bot_description/meshes/STL/upper_side_leg.stl; visual mesh filename=package://echo_bot_description/meshes/DAE/upper_side_leg.dae
- link wheel_left_link: mass 0.039831 -> None; geometry collision cylinder length=0.02 radius=0.029; visual mesh filename=package://echo_bot_description/meshes/DAE/tyre.dae
- link wheel_right_link: mass 0.039831 -> None; geometry collision cylinder length=0.02 radius=0.029; visual mesh filename=package://echo_bot_description/meshes/DAE/tyre.dae
Joints:
- removed joint side_leg_left_joint
- removed joint side_leg_right_joint
- joint base_link_joint: origin xyz=0 0 0.20 -> xyz=0 0 0.090; parent world -> base_footprint
- joint lower_leg_left: limit lower=0.0 upper=1.16465824189 effort=0 velocity=0 -> lower=0.0 upper=1.16465824189 effort=30 velocity=3.14159274
- joint lower_leg_right: limit lower=0.0 upper=1.16465824189 effort=0 velocity=0 -> lower=0.0 upper=1.16465824189 effort=30 velocity=3.14159274
- joint upper_leg_left_joint: limit lower=0.0 upper=-0.52359879 effort=0 velocity=0 -> lower=0.0 upper=-0.52359879 effort=30 velocity=3.14159274
- joint upper_leg_right_joint: limit lower=0.0 upper=-0.52359879 effort=0 velocity=0 -> lower=0.0 upper=-0.52359879 effort=30 velocity=3.14159274
- joint upper_side_leg_left: limit lower=0.0 upper=-1.12975165589 effort=0 velocity=0 -> lower=0.0 upper=-1.12975165589 effort=30 velocity=3.14159274
- joint upper_side_leg_right: limit lower=0.0 upper=-1.12975165589 effort=0 velocity=0 -> lower=0.0 upper=-1.12975165589 effort=30 velocity=3.14159274
- joint wheel_left_joint: limit (none) -> effort=0.4 velocity=12.0
- joint wheel_right_joint: limit (none) -> effort=0.4 velocity=12.0

File: echo_bot_description/urdf/wheel/echo_bot_wheel.gazebo.xacro (robot description, xacro)
@@ -4,6 +4,10 @@
     <gazebo reference="wheel_${prefix}_link">
       <selfCollide>true</selfCollide>
-      <mu1 value="0.8" />
-      <mu2 value="0.8" />
+      <!-- <mu1 value="0.8" />
+      <mu2 value="0.8" /> -->
+      <mu1 value="2.5" />
+      <mu2 value="2.5" />
+      <kp value="50000" />
+      <kd value="10" />
     </gazebo>
   </xacro:macro>

File: echo_bot_description/urdf/wheel/echo_bot_wheel.transmission.xacro (robot description, xacro)
@@ -9,5 +9,5 @@
       <actuator name="wheel_${prefix}_motor">
         <hardwareInterface>hardware_interface/VelocityJointInterface</hardwareInterface>
-        <mechanicalReduction>30</mechanicalReduction>
+        <mechanicalReduction>1</mechanicalReduction>
       </actuator>
     </transmission>

File: echo_bot_description/urdf/wheel/echo_bot_wheel.urdf.xacro (robot description, xacro)
@@ -1,15 +1,18 @@
 <?xml version="1.0"?>
 <robot xmlns:xacro="http://ros.org/wiki/xacro">
-<xacro:include filename="$(find echo_bot_description)/urdf/wheel/echo_bot_wheel.transmission.xacro"/>
-<xacro:include filename="$(find echo_bot_description)/urdf/wheel/echo_bot_wheel.gazebo.xacro"/>
-  <!-- == Material == -->
-  <material name="wheel_color">
-    <color rgba="0.3 0.3 0.3 1"/>
-  </material>
+  <xacro:include filename="$(find echo_bot_description)/urdf/wheel/echo_bot_wheel.transmission.xacro"/>
+  <xacro:include filename="$(find echo_bot_description)/urdf/wheel/echo_bot_wheel.gazebo.xacro"/>
+  <property name="wheel_radius" value="0.029"/>
+  <property name="wheel_length" value="0.012"/>
+  <property name="wheel_mass" value="0.039831"/>
+  <xacro:macro name="cylinder_inertial" params="mass radius length">
+    <mass value="${mass}"/>
+    <inertia  ixx="${((radius*radius)/4 + (length*length)/12)*mass}" ixy="0" ixz="0"
+              iyy="${((radius*radius)/4 + (length*length)/12)*mass}" iyz="0"
+              izz="${(mass*radius*radius)/2}" />
+  </xacro:macro>
   <xacro:macro name="wheel_v0" params="prefix parent *joint_origin *joint_axis">
     <link name="wheel_${prefix}_link">
       <visual>
-        <origin rpy="0 0 0"/>
-        <material name="wheel_color"/>
         <geometry>
           <mesh filename="package://echo_bot_description/meshes/DAE/tyre.dae"/>
@@ -17,15 +20,14 @@
       </visual>
       <collision>
-        <origin rpy="0 0 0"/>
+        <!-- <origin xyz="0 -0.003 0" rpy="${-M_PI/2} 0 0"/> -->
+        <origin xyz="0 0 0" rpy="0 0 0"/>
         <geometry>
-          <mesh filename="package://echo_bot_description/meshes/STL/tyre.stl"/>
+          <cylinder radius="${wheel_radius}" length="${wheel_length}"/>
         </geometry>
       </collision>
       <inertial>
-        <mass value="0.039831"/>
         <origin xyz="0.0 0.0 0.0" rpy="0 0 0"/>
-        <inertia  ixx="0.000008" ixy="0.0" ixz="0.0"
-                  iyy="0.000008" iyz="0.0"
-                  izz="0.000015"/>
+        <cylinder_inertial  mass="${wheel_mass}"
+                            radius="${wheel_radius}" length="${wheel_length}"/>
       </inertial>
     </link>
@@ -35,4 +37,6 @@
       <child link="wheel_${prefix}_link"/>
       <insert_block name="joint_axis"/>
+      <limit velocity="12.0" effort="0.4" />
+      <dynamics damping="0.1"/>
     </joint>
   </xacro:macro>
