Commit message: rename

File: echo_bot_description/robots/echo_bot.urdf.xacro (robot description, xacro)
@@ -15,9 +15,10 @@
     <origin xyz="0.0 0.0475 0.0" rpy="0.0 ${M_PI*160/180} 0.0"/>
   </xacro:left_leg_v0>
+  <!-- == left_wheel == -->
   <xacro:wheel_v0 prefix="left" parent="lower_leg_L">
     <origin xyz="0.1 0.0305 0.0" rpy="${-M_PI/2} 0.0 0.0"/>
     <axis xyz="0 0 1"/>
   </xacro:wheel_v0>
-  <xacro:joint_velocity_trans_v0 prefix="left"/>
+  <xacro:wheel_trans_v0 prefix="left"/>
   <!-- == right_leg == -->
   <!-- <xacro:include filename="$(find echo_bot_description)/urdf/leg/echo_bot_right_leg.urdf.xacro"/> -->
@@ -26,9 +27,11 @@
   <gazebo>
     <plugin name="gazebo_ros_control" filename="libgazebo_ros_control.so">
-      <robotNamespace>echo_bot</robotNamespace>
+      <!-- <robotNamespace>echo_bot</robotNamespace> -->
     </plugin>
   </gazebo>
   <!-- Base -->
   <xacro:base_gazebo_v0/>
+  <!-- Left leg -->
+  <xacro:left_leg_gazebo_v0/>
   <!-- Wheel -->
   <xacro:wheel_gazebo_v0 prefix="left"/>

File: echo_bot_description/robots/test.urdf (robot description, URDF)
Before this commit: robot echo_bot, 6 links, 5 joints
Links:
- removed link wheel_left
- added link wheel_left_link, mass 13.25; collision mesh filename=package://echo_bot_description/meshes/DAE/tyre.dae; visual mesh filename=package://echo_bot_description/meshes/STL/tyre.stl
- link base_link: geometry collision mesh filename=package://echo_bot_description/meshes/DAE/body.dae; visual mesh filename=package://echo_bot_description/meshes/STL/body.stl
- link lower_leg_L: geometry collision mesh filename=package://echo_bot_description/meshes/DAE/lower_leg.dae; visual mesh filename=package://echo_bot_description/meshes/STL/lower_leg.stl
- link upper_leg_L: geometry collision mesh filename=package://echo_bot_description/meshes/DAE/upper_leg.dae; visual mesh filename=package://echo_bot_description/meshes/STL/upper_leg.stl
- link upper_side_leg_L: geometry collision mesh filename=package://echo_bot_description/meshes/DAE/upper_side_leg.dae; visual mesh filename=package://echo_bot_description/meshes/STL/upper_side_leg.stl
Joints:
- removed joint wheel_left
- added joint wheel_left_joint: type continuous, parent lower_leg_L, child wheel_left_link, origin xyz=0.1 0.0305 0.0 rpy=-1.57079637 0.0 0.0, axis 0 0 1

Commit message: rename "L" to "left"

File: echo_bot_description/robots/echo_bot.urdf.xacro (robot description, xacro)
@@ -16,5 +16,5 @@
   </xacro:left_leg_v0>
   <!-- == left_wheel == -->
-  <xacro:wheel_v0 prefix="left" parent="lower_leg_L">
+  <xacro:wheel_v0 prefix="left" parent="lower_leg_left">
     <origin xyz="0.1 0.0305 0.0" rpy="${-M_PI/2} 0.0 0.0"/>
     <axis xyz="0 0 1"/>

File: echo_bot_description/urdf/leg/echo_bot_left_leg.urdf.xacro (robot description, xacro)
@@ -1,4 +1,5 @@
 <?xml version="1.0"?>
-<robot name="echo_bot" xmlns:xacro="http://ros.org/wiki/xacro">
+<robot xmlns:xacro="http://ros.org/wiki/xacro">
+  <xacro:include filename="$(find echo_bot_description)/urdf/leg/echo_bot_left_leg.gazebo.xacro"/>
   <!-- == Material == -->
   <material name="leg_color_0">
@@ -6,89 +7,89 @@
   </material>
   <xacro:macro name="left_leg_v0" params="parent *joint_origin">
-  <!-- Link -->
-  <link name="upper_leg_L">
-    <visual>
-      <origin rpy="0 0 0"/>
-      <material name="leg_color_0"/>
-      <geometry>
-        <mesh filename="package://echo_bot_description/meshes/STL/upper_leg.stl"/>
-      </geometry>
-    </visual>
-    <collision>
-      <origin rpy="0 0 0"/>
-      <geometry>
-        <mesh filename="package://echo_bot_description/meshes/STL/upper_leg.stl"/>
-      </geometry>
-    </collision>
-    <inertial>
-      <mass value="13.25" />
-      <origin xyz="0.0 0.0 0.0" rpy="0 0 0" />
-      <inertia ixx="0.2015" ixy="0.0" ixz="0.0" iyy="0.265" iyz="0.0" izz="0.2015" />
-    </inertial>
-  </link>
-  <link name="lower_leg_L">
-    <visual>
-      <origin rpy="0 0 0"/>
-      <material name="leg_color_0"/>
-      <geometry>
-        <mesh filename="package://echo_bot_description/meshes/STL/lower_leg.stl"/>
-      </geometry>
-    </visual>
-    <collision>
-      <origin rpy="0 0 0"/>
-      <geometry>
-        <mesh filename="package://echo_bot_description/meshes/STL/lower_leg.stl"/>
-      </geometry>
-    </collision>
-    <inertial>
-      <mass value="13.25" />
-      <origin xyz="0.0 0.0 0.0" rpy="0 0 0" />
-      <inertia ixx="0.2015" ixy="0.0" ixz="0.0" iyy="0.265" iyz="0.0" izz="0.2015" />
-    </inertial>
-  </link>
-  <link name="upper_side_leg_L">
-    <visual>
-      <origin rpy="0 0 0"/>
-      <material name="leg_color_0"/>
-      <geometry>
-        <mesh filename="package://echo_bot_description/meshes/STL/upper_side_leg.stl"/>
-      </geometry>
-    </visual>
-    <collision>
-      <origin rpy="0 0 0"/>
-      <geometry>
-        <mesh filename="package://echo_bot_description/meshes/STL/upper_side_leg.stl"/>
-      </geometry>
-    </collision>
-    <inertial>
-      <mass value="13.25" />
-      <origin xyz="0.0 0.0 0.0" rpy="0 0 0" />
-      <inertia ixx="0.2015" ixy="0.0" ixz="0.0" iyy="0.265" iyz="0.0" izz="0.2015" />
-    </inertial>
-  </link>
-  <!-- Joint -->
-  <joint name="upper_leg_L" type="revolute">
-    <insert_block name="joint_origin"/>
-    <parent link="${parent}" />
-    <child link="upper_leg_L" />
-    <axis xyz="0 1 0"/>
-    <limit lower="0.0" upper="${-M_PI*30/180}" effort="0" velocity="0"/>
-  </joint>
-  <joint name="lower_leg_L" type="revolute">
-    <origin xyz="0.1 0.0 0.0" rpy="0.0 ${-M_PI*144.47/180} 0.0" />
-    <parent link="upper_leg_L" />
-    <child link="lower_leg_L" />
-    <axis xyz="0 1 0"/>
-    <limit lower="0.0" upper="${M_PI*66.73/180}" effort="0" velocity="0"/>
-    <mimic joint="upper_leg_L" multiplier="-2.186" offset="-0.02025"/>
-  </joint>
-  <joint name="upper_side_leg_L" type="revolute">
-    <origin xyz="-0.025 0.0 0.0" rpy="0.0 ${-M_PI*54.22/180} 0.0" />
-    <parent link="lower_leg_L" />
-    <child link="upper_side_leg_L" />
-    <axis xyz="0 1 0"/>
-    <limit lower="0.0" upper="${-M_PI*64.73/180}" effort="0" velocity="0"/>
-    <mimic joint="upper_leg_L" multiplier="2.123937" offset="0.003625"/>
-  </joint>
+    <!-- Link -->
+    <link name="upper_leg_left">
+      <visual>
+        <origin rpy="0 0 0"/>
+        <material name="leg_color_0"/>
+        <geometry>
+          <mesh filename="package://echo_bot_description/meshes/STL/upper_leg.stl"/>
+        </geometry>
+      </visual>
+      <collision>
+        <origin rpy="0 0 0"/>
+        <geometry>
+          <mesh filename="package://echo_bot_description/meshes/DAE/upper_leg.dae"/>
+        </geometry>
+      </collision>
+      <inertial>
+        <mass value="13.25" />
+        <origin xyz="0.0 0.0 0.0" rpy="0 0 0" />
+        <inertia ixx="0.2015" ixy="0.0" ixz="0.0" iyy="0.265" iyz="0.0" izz="0.2015" />
+      </inertial>
+    </link>
+    <link name="lower_leg_left">
+      <visual>
+        <origin rpy="0 0 0"/>
+        <material name="leg_color_0"/>
+        <geometry>
+          <mesh filename="package://echo_bot_description/meshes/STL/lower_leg.stl"/>
+        </geometry>
+      </visual>
+      <collision>
+        <origin rpy="0 0 0"/>
+        <geometry>
+          <mesh filename="package://echo_bot_description/meshes/DAE/lower_leg.dae"/>
+        </geometry>
+      </collision>
+      <inertial>
+        <mass value="13.25" />
+        <origin xyz="0.0 0.0 0.0" rpy="0 0 0" />
+        <inertia ixx="0.2015" ixy="0.0" ixz="0.0" iyy="0.265" iyz="0.0" izz="0.2015" />
+      </inertial>
+    </link>
+    <link name="upper_side_leg_left">
+      <visual>
+        <origin rpy="0 0 0"/>
+        <material name="leg_color_0"/>
+        <geometry>
+          <mesh filename="package://echo_bot_description/meshes/STL/upper_side_leg.stl"/>
+        </geometry>
+      </visual>
+      <collision>
+        <origin rpy="0 0 0"/>
+        <geometry>
+          <mesh filename="package://echo_bot_description/meshes/DAE/upper_side_leg.dae"/>
+        </geometry>
+      </collision>
+      <inertial>
+        <mass value="13.25" />
+        <origin xyz="0.0 0.0 0.0" rpy="0 0 0" />
+        <inertia ixx="0.2015" ixy="0.0" ixz="0.0" iyy="0.265" iyz="0.0" izz="0.2015" />
+      </inertial>
+    </link>
+    <!-- Joint -->
+    <joint name="upper_leg_left" type="revolute">
+      <insert_block name="joint_origin"/>
+      <parent link="${parent}" />
+      <child link="upper_leg_left" />
+      <axis xyz="0 1 0"/>
+      <limit lower="0.0" upper="${-M_PI*30/180}" effort="0" velocity="0"/>
+    </joint>
+    <joint name="lower_leg_left" type="revolute">
+      <origin xyz="0.1 0.0 0.0" rpy="0.0 ${-M_PI*144.47/180} 0.0" />
+      <parent link="upper_leg_left" />
+      <child link="lower_leg_left" />
+      <axis xyz="0 1 0"/>
+      <limit lower="0.0" upper="${M_PI*66.73/180}" effort="0" velocity="0"/>
+      <mimic joint="upper_leg_left" multiplier="-2.186" offset="-0.02025"/>
+    </joint>
+    <joint name="upper_side_leg_left" type="revolute">
+      <origin xyz="-0.025 0.0 0.0" rpy="0.0 ${-M_PI*54.22/180} 0.0" />
+      <parent link="lower_leg_left" />
+      <child link="upper_side_leg_left" />
+      <axis xyz="0 1 0"/>
+      <limit lower="0.0" upper="${-M_PI*64.73/180}" effort="0" velocity="0"/>
+      <mimic joint="upper_leg_left" multiplier="2.123937" offset="0.003625"/>
+    </joint>
   </xacro:macro>
 </robot>

File: echo_bot_description/urdf/wheel/echo_bot_wheel.urdf.xacro (robot description, xacro)
@@ -1,4 +1,4 @@
 <?xml version="1.0"?>
-<robot name="echo_bot" xmlns:xacro="http://ros.org/wiki/xacro">
+<robot xmlns:xacro="http://ros.org/wiki/xacro">
 <xacro:include filename="$(find echo_bot_description)/urdf/wheel/echo_bot_wheel.transmission.xacro"/>
 <xacro:include filename="$(find echo_bot_description)/urdf/wheel/echo_bot_wheel.gazebo.xacro"/>
@@ -8,5 +8,5 @@
   </material>
   <xacro:macro name="wheel_v0" params="prefix parent *joint_origin *joint_axis">
-    <link name="wheel_${prefix}">
+    <link name="wheel_${prefix}_link">
       <visual>
         <origin rpy="0 0 0"/>
@@ -19,5 +19,5 @@
         <origin rpy="0 0 0"/>
         <geometry>
-          <mesh filename="package://echo_bot_description/meshes/STL/tyre.stl"/>
+          <mesh filename="package://echo_bot_description/meshes/DAE/tyre.dae"/>
         </geometry>
       </collision>
@@ -28,8 +28,8 @@
       </inertial>
     </link>
-    <joint name="wheel_${prefix}" type="continuous">
+    <joint name="wheel_${prefix}_joint" type="continuous">
       <insert_block name="joint_origin"/>
       <parent link="${parent}" />
-      <child link="wheel_${prefix}"/>
+      <child link="wheel_${prefix}_link"/>
       <insert_block name="joint_axis"/>
     </joint>

Commit message: add right leg model & correct parameters

File: echo_bot_description/robots/echo_bot.urdf.xacro (robot description, xacro)
@@ -11,7 +11,13 @@
   </xacro:base_v0>
   <!-- == left_leg == -->
-  <xacro:left_leg_v0 parent="base_link">
+  <xacro:leg_v0 parent="base_link" prefix="left">
     <origin xyz="0.0 0.0475 0.0" rpy="0.0 ${M_PI*160/180} 0.0"/>
-  </xacro:left_leg_v0>
+  </xacro:leg_v0>
+  <xacro:leg_trans_v0 prefix="left"/>
+  <!-- == right_leg == -->
+  <xacro:leg_v0 parent="base_link" prefix="right">
+    <origin xyz="0.0 -0.0475 0.0" rpy="0.0 ${M_PI*160/180} 0.0"/>
+  </xacro:leg_v0>
+  <xacro:leg_trans_v0 prefix="right"/>
   <!-- == left_wheel == -->
   <xacro:wheel_v0 prefix="left" parent="lower_leg_left">
@@ -20,17 +26,27 @@
   </xacro:wheel_v0>
   <xacro:wheel_trans_v0 prefix="left"/>
-  <!-- == right_leg == -->
+  <!-- == right_wheel == -->
+  <xacro:wheel_v0 prefix="right" parent="lower_leg_right">
+    <origin xyz="0.1 -0.0305 0.0" rpy="${-M_PI/2} 0.0 0.0"/>
+    <axis xyz="0 0 1"/>
+  </xacro:wheel_v0>
+  <xacro:wheel_trans_v0 prefix="right"/>
   <!-- == Sensor == -->
   <!-- == Gazebo == -->
   <gazebo>
     <plugin name="gazebo_ros_control" filename="libgazebo_ros_control.so">
-      <!-- <robotNamespace>echo_bot</robotNamespace> -->
+      <robotNamespace>echo_bot</robotNamespace>
     </plugin>
   </gazebo>
+  <plugin name="joint_state_publisher" filename="libgazebo_ros_joint_state_publisher.so">
+    <jointName>upper_leg_left_joint, upper_leg_right_joint, wheel_left_joint, wheel_right_joint</jointName>
+  </plugin>
   <!-- Base -->
   <xacro:base_gazebo_v0/>
   <!-- Left leg -->
-  <xacro:left_leg_gazebo_v0/>
+  <xacro:leg_gazebo_v0 prefix="left"/>
+  <xacro:leg_gazebo_v0 prefix="right"/>
   <!-- Wheel -->
   <xacro:wheel_gazebo_v0 prefix="left"/>
+  <xacro:wheel_gazebo_v0 prefix="right"/>
 </robot>

File: echo_bot_description/robots/test.urdf (robot description, URDF)
Before this commit: robot echo_bot, 6 links, 5 joints
Links:
- removed link lower_leg_L
- removed link upper_leg_L
- removed link upper_side_leg_L
- added link lower_leg_left, mass 13.25; collision mesh filename=package://echo_bot_description/meshes/DAE/lower_leg.dae; visual mesh filename=package://echo_bot_description/meshes/STL/lower_leg.stl
- added link lower_leg_right, mass 13.25; collision mesh filename=package://echo_bot_description/meshes/DAE/lower_leg.dae; visual mesh filename=package://echo_bot_description/meshes/STL/lower_leg.stl
- added link upper_leg_left, mass 13.25; collision mesh filename=package://echo_bot_description/meshes/DAE/upper_leg.dae; visual mesh filename=package://echo_bot_description/meshes/STL/upper_leg.stl
- added link upper_leg_right, mass 13.25; collision mesh filename=package://echo_bot_description/meshes/DAE/upper_leg.dae; visual mesh filename=package://echo_bot_description/meshes/STL/upper_leg.stl
- added link upper_side_leg_left, mass 13.25; collision mesh filename=package://echo_bot_description/meshes/DAE/upper_side_leg.dae; visual mesh filename=package://echo_bot_description/meshes/STL/upper_side_leg.stl
- added link upper_side_leg_right, mass 13.25; collision mesh filename=package://echo_bot_description/meshes/DAE/upper_side_leg.dae; visual mesh filename=package://echo_bot_description/meshes/STL/upper_side_leg.stl
- added link wheel_right_link, mass 13.25; collision mesh filename=package://echo_bot_description/meshes/DAE/tyre.dae; visual mesh filename=package://echo_bot_description/meshes/STL/tyre.stl
- link base_link: mass 1e-06 -> 1e-05
Joints:
- removed joint lower_leg_L
- removed joint upper_leg_L
- removed joint upper_side_leg_L
- added joint lower_leg_left: type revolute, parent upper_leg_left, child lower_leg_left, origin xyz=0.1 0.0 0.0 rpy=0.0 -2.52147723971 0.0, axis 0 1 0, limit lower=0.0 upper=1.16465824189 effort=0 velocity=0, mimic joint=upper_leg_left_joint multiplier=-2.186 offset=-0.02025
- added joint lower_leg_right: type revolute, parent upper_leg_right, child lower_leg_right, origin xyz=0.1 0.0 0.0 rpy=0.0 -2.52147723971 0.0, axis 0 1 0, limit lower=0.0 upper=1.16465824189 effort=0 velocity=0, mimic joint=upper_leg_right_joint multiplier=-2.186 offset=-0.02025
- added joint upper_leg_left_joint: type revolute, parent base_link, child upper_leg_left, origin xyz=0.0 0.0475 0.0 rpy=0.0 2.79252688 0.0, axis 0 1 0, limit lower=0.0 upper=-0.52359879 effort=0 velocity=0
- added joint upper_leg_right_joint: type revolute, parent base_link, child upper_leg_right, origin xyz=0.0 -0.0475 0.0 rpy=0.0 2.79252688 0.0, axis 0 1 0, limit lower=0.0 upper=-0.52359879 effort=0 velocity=0
- added joint upper_side_leg_left: type revolute, parent lower_leg_left, child upper_side_leg_left, origin xyz=-0.025 0.0 0.0 rpy=0.0 -0.94631754646 0.0, axis 0 1 0, limit lower=0.0 upper=-1.12975165589 effort=0 velocity=0, mimic joint=upper_leg_left_joint multiplier=2.123937 offset=0.003625
- added joint upper_side_leg_right: type revolute, parent lower_leg_right, child upper_side_leg_right, origin xyz=-0.025 0.0 0.0 rpy=0.0 -0.94631754646 0.0, axis 0 1 0, limit lower=0.0 upper=-1.12975165589 effort=0 velocity=0, mimic joint=upper_leg_right_joint multiplier=2.123937 offset=0.003625
- added joint wheel_right_joint: type continuous, parent lower_leg_right, child wheel_right_link, origin xyz=0.1 -0.0305 0.0 rpy=-1.57079637 0.0 0.0, axis 0 0 1
- joint wheel_left_joint: parent lower_leg_L -> lower_leg_left

File: echo_bot_description/urdf/base/echo_bot_base.urdf.xacro (robot description, xacro)
@@ -22,7 +22,9 @@
       </collision>
       <inertial>
-        <mass value="1e-05" />
+        <mass value="2.915" />
         <origin xyz="0 0 0" rpy="0 0 0" />
-        <inertia ixx="1.0" ixy="0.0" ixz="0.0" iyy="1.0" iyz="0.0" izz="1.0" />
+        <inertia  ixx="0.006" ixy="0.0" ixz="0.002"
+                  iyy="0.008" iyz="0.0"
+                  izz="0.009"/>
       </inertial>
     </link>

File: echo_bot_description/urdf/leg/echo_bot_left_leg.urdf.xacro (robot description, xacro)
@@ -1,12 +1,13 @@
 <?xml version="1.0"?>
 <robot xmlns:xacro="http://ros.org/wiki/xacro">
-  <xacro:include filename="$(find echo_bot_description)/urdf/leg/echo_bot_left_leg.gazebo.xacro"/>
+  <xacro:include filename="$(find echo_bot_description)/urdf/leg/echo_bot_leg.transmission.xacro"/>
+  <xacro:include filename="$(find echo_bot_description)/urdf/leg/echo_bot_leg.gazebo.xacro"/>
   <!-- == Material == -->
   <material name="leg_color_0">
     <color rgba="0.3 0.3 0.3 1"/>
   </material>
-  <xacro:macro name="left_leg_v0" params="parent *joint_origin">
+  <xacro:macro name="leg_v0" params="parent prefix *joint_origin">
     <!-- Link -->
-    <link name="upper_leg_left">
+    <link name="upper_leg_${prefix}">
       <visual>
         <origin rpy="0 0 0"/>
@@ -23,15 +24,17 @@
       </collision>
       <inertial>
-        <mass value="13.25" />
+        <mass value="0.109" />
         <origin xyz="0.0 0.0 0.0" rpy="0 0 0" />
-        <inertia ixx="0.2015" ixy="0.0" ixz="0.0" iyy="0.265" iyz="0.0" izz="0.2015" />
+        <inertia  ixx="0.000068" ixy="0.0" ixz="0.0"
+                  iyy="0.000086" iyz="0.0"
+                  izz="0.000136" />
       </inertial>
     </link>
-    <link name="lower_leg_left">
+    <link name="lower_leg_${prefix}">
       <visual>
         <origin rpy="0 0 0"/>
         <material name="leg_color_0"/>
         <geometry>
-          <mesh filename="package://echo_bot_description/meshes/STL/lower_leg.stl"/>
+          <mesh filename="package://echo_bot_description/meshes/STL/lower_leg_${prefix}.stl"/>
         </geometry>
       </visual>
@@ -39,14 +42,16 @@
         <origin rpy="0 0 0"/>
         <geometry>
-          <mesh filename="package://echo_bot_description/meshes/DAE/lower_leg.dae"/>
+          <mesh filename="package://echo_bot_description/meshes/DAE/lower_leg_${prefix}.dae"/>
         </geometry>
       </collision>
       <inertial>
-        <mass value="13.25" />
+        <mass value="0.152994" />
         <origin xyz="0.0 0.0 0.0" rpy="0 0 0" />
-        <inertia ixx="0.2015" ixy="0.0" ixz="0.0" iyy="0.265" iyz="0.0" izz="0.2015" />
+        <inertia  ixx="0.000046" ixy="-0.000012" ixz="-0.000001"
+                  iyy="0.000243" iyz="0.0"
+                  izz="0.000238" />
       </inertial>
     </link>
-    <link name="upper_side_leg_left">
+    <link name="upper_side_leg_${prefix}">
       <visual>
         <origin rpy="0 0 0"/>
@@ -63,32 +68,34 @@
       </collision>
       <inertial>
-        <mass value="13.25" />
-        <origin xyz="0.0 0.0 0.0" rpy="0 0 0" />
-        <inertia ixx="0.2015" ixy="0.0" ixz="0.0" iyy="0.265" iyz="0.0" izz="0.2015" />
+        <mass value="0.041157"/>
+        <origin xyz="0.0 0.0 0.0" rpy="0 0 0"/>
+        <inertia  ixx="0.000003" ixy="0.0" ixz="0.0"
+                  iyy="0.000043" iyz="0.0"
+                  izz="0.000043"/>
       </inertial>
     </link>
     <!-- Joint -->
-    <joint name="upper_leg_left" type="revolute">
+    <joint name="upper_leg_${prefix}_joint" type="revolute">
       <insert_block name="joint_origin"/>
       <parent link="${parent}" />
-      <child link="upper_leg_left" />
+      <child link="upper_leg_${prefix}" />
       <axis xyz="0 1 0"/>
       <limit lower="0.0" upper="${-M_PI*30/180}" effort="0" velocity="0"/>
     </joint>
-    <joint name="lower_leg_left" type="revolute">
+    <joint name="lower_leg_${prefix}" type="revolute">
       <origin xyz="0.1 0.0 0.0" rpy="0.0 ${-M_PI*144.47/180} 0.0" />
-      <parent link="upper_leg_left" />
-      <child link="lower_leg_left" />
+      <parent link="upper_leg_${prefix}" />
+      <child link="lower_leg_${prefix}" />
       <axis xyz="0 1 0"/>
       <limit lower="0.0" upper="${M_PI*66.73/180}" effort="0" velocity="0"/>
-      <mimic joint="upper_leg_left" multiplier="-2.186" offset="-0.02025"/>
+      <mimic joint="upper_leg_${prefix}_joint" multiplier="-2.186" offset="-0.02025"/>
     </joint>
-    <joint name="upper_side_leg_left" type="revolute">
+    <joint name="upper_side_leg_${prefix}" type="revolute">
       <origin xyz="-0.025 0.0 0.0" rpy="0.0 ${-M_PI*54.22/180} 0.0" />
-      <parent link="lower_leg_left" />
-      <child link="upper_side_leg_left" />
+      <parent link="lower_leg_${prefix}" />
+      <child link="upper_side_leg_${prefix}" />
       <axis xyz="0 1 0"/>
       <limit lower="0.0" upper="${-M_PI*64.73/180}" effort="0" velocity="0"/>
-      <mimic joint="upper_leg_left" multiplier="2.123937" offset="0.003625"/>
+      <mimic joint="upper_leg_${prefix}_joint" multiplier="2.123937" offset="0.003625"/>
     </joint>
   </xacro:macro>

File: echo_bot_description/urdf/leg/echo_bot_leg.gazebo.xacro (robot description, xacro)
@@ -1,16 +1,16 @@
 <?xml version="1.0"?>
 <robot name="echo_bot" xmlns:xacro="http://ros.org/wiki/xacro">
-  <xacro:macro name="left_leg_gazebo_v0">
-    <gazebo reference="upper_leg_left">
+  <xacro:macro name="leg_gazebo_v0" params="prefix">
+    <gazebo reference="upper_leg_${prefix}">
       <selfCollide>true</selfCollide>
       <mu1 value="0.8" />
       <mu2 value="0.8" />
     </gazebo>
-    <gazebo reference="lower_leg_left">
+    <gazebo reference="lower_leg_${prefix}">
       <selfCollide>true</selfCollide>
       <mu1 value="0.8" />
       <mu2 value="0.8" />
     </gazebo>
-    <gazebo reference="upper_side_leg_left">
+    <gazebo reference="upper_side_leg_${prefix}">
       <selfCollide>true</selfCollide>
       <mu1 value="0.8" />

File: echo_bot_description/urdf/wheel/echo_bot_wheel.gazebo.xacro (robot description, xacro)
@@ -4,6 +4,6 @@
     <gazebo reference="wheel_${prefix}_link">
       <selfCollide>true</selfCollide>
-      <mu1 value="0.8" />
-      <mu2 value="0.8" />
+      <mu1 value="0.05" />
+      <mu2 value="0.05" />
     </gazebo>
   </xacro:macro>

File: echo_bot_description/urdf/wheel/echo_bot_wheel.urdf.xacro (robot description, xacro)
@@ -23,7 +23,9 @@
       </collision>
       <inertial>
-        <mass value="13.25" />
-        <origin xyz="0.0 0.0 0.0" rpy="0 0 0" />
-        <inertia ixx="0.2015" ixy="0.0" ixz="0.0" iyy="0.265" iyz="0.0" izz="0.2015" />
+        <mass value="0.039831"/>
+        <origin xyz="0.0 0.0 0.0" rpy="0 0 0"/>
+        <inertia  ixx="0.000008" ixy="0.0" ixz="0.0"
+                  iyy="0.000008" iyz="0.0"
+                  izz="0.000015"/>
       </inertial>
     </link>
