Commit message: ros_controller work done

File: echo_bot_description/robots/echo_bot.urdf.xacro (robot description, xacro)
@@ -22,5 +22,5 @@
   <!-- == left_wheel == -->
   <xacro:wheel_v0 prefix="left" parent="lower_leg_left">
-    <origin xyz="0.1 0.0305 0.0" rpy="${-M_PI/2} 0.0 0.0"/>
+    <origin xyz="0.1 0.0305 0.0" rpy="${-M_PI/2} 0.0 ${M_PI}"/>
     <axis xyz="0 0 1"/>
   </xacro:wheel_v0>
@@ -37,4 +37,6 @@
     <plugin name="gazebo_ros_control" filename="libgazebo_ros_control.so">
       <robotNamespace>echo_bot</robotNamespace>
+      <robotSimType>gazebo_ros_control/DefaultRobotHWSim</robotSimType>
+      <legacyModeNS>true</legacyModeNS>
     </plugin>
   </gazebo>
@@ -44,7 +46,25 @@
   <!-- Base -->
   <xacro:base_gazebo_v0/>
-  <!-- Left leg -->
+  <!-- leg -->
   <xacro:leg_gazebo_v0 prefix="left"/>
   <xacro:leg_gazebo_v0 prefix="right"/>
+  <gazebo>
+    <plugin name="left_leg_ClosedLoopPlugin" filename="libpegasus_gazebo_closed_loop_plugin.so">
+      <joint>base_back_joint</joint>
+      <child>side_leg_left</child>
+      <parent>upper_side_leg_left</parent>
+      <position>0.1 0.0 0.0</position>
+      <rotation>0.00 -0.00 0.00</rotation>
+    </plugin>
+  </gazebo>
+  <gazebo>
+    <plugin name="right_leg_ClosedLoopPlugin" filename="libpegasus_gazebo_closed_loop_plugin.so">
+      <joint>base_back_joint</joint>
+      <child>side_leg_right</child>
+      <parent>upper_side_leg_right</parent>
+      <position>0.1 0.0 0.0</position>
+      <rotation>0.00 -0.00 0.00</rotation>
+    </plugin>
+  </gazebo>
   <!-- Wheel -->
   <xacro:wheel_gazebo_v0 prefix="left"/>

File: echo_bot_description/urdf/base/echo_bot_base.urdf.xacro (robot description, xacro)
@@ -29,4 +29,6 @@
       </inertial>
     </link>
+    <link name="side_leg_left"/>
+    <link name="side_leg_right"/>
     <joint name="base_link_joint" type="fixed">
       <insert_block name="joint_origin"/>
@@ -34,4 +36,14 @@
       <child link="base_link"/>
     </joint>
+    <joint name="side_leg_left_joint" type="fixed">
+      <origin xyz="-0.04 0.0475 0.035" rpy="0 0 0"/>
+      <parent link="base_link"/>
+      <child link="side_leg_left"/>
+    </joint>
+    <joint name="side_leg_right_joint" type="fixed">
+      <origin xyz="-0.04 -0.0475 0.035" rpy="0 0 0"/>
+      <parent link="base_link"/>
+      <child link="side_leg_right"/>
+    </joint>
   </xacro:macro>
 </robot>

File: echo_bot_description/urdf/leg/echo_bot_leg.transmission.xacro (robot description, xacro)
@@ -5,7 +5,8 @@
       <type>transmission_interface/SimpleTransmission</type>
       <joint name="upper_leg_${prefix}_joint">
-        <hardwareInterface>hardware_interface/PositionJointInterface</hardwareInterface>
+        <hardwareInterface>hardware_interface/EffortJointInterface</hardwareInterface>
       </joint>
       <actuator name="leg_${prefix}_motor">
+        <hardwareInterface>hardware_interface/EffortJointInterface</hardwareInterface>
         <mechanicalReduction>1</mechanicalReduction>
       </actuator>

Commit message: JointTrajectoryController実装（lower_leg_leftしか動かない。）

File: echo_bot_description/robots/echo_bot.urdf.xacro (robot description, xacro)
@@ -10,14 +10,16 @@
   <origin xyz="0 0 0.090"/>
   </xacro:base_v0>
+  <!-- <link name="world"/>
+  <xacro:base_v0 parent="world">
+  <origin xyz="0 0 0.20"/>
+  </xacro:base_v0> -->
   <!-- == left_leg == -->
   <xacro:leg_v0 parent="base_link" prefix="left">
     <origin xyz="0.0 0.0475 0.0" rpy="0.0 ${M_PI*160/180} 0.0"/>
   </xacro:leg_v0>
-  <xacro:leg_trans_v0 prefix="left"/>
   <!-- == right_leg == -->
   <xacro:leg_v0 parent="base_link" prefix="right">
     <origin xyz="0.0 -0.0475 0.0" rpy="0.0 ${M_PI*160/180} 0.0"/>
   </xacro:leg_v0>
-  <xacro:leg_trans_v0 prefix="right"/>
   <!-- == left_wheel == -->
   <xacro:wheel_v0 prefix="left" parent="lower_leg_left">
@@ -49,10 +51,10 @@
   <xacro:leg_gazebo_v0 prefix="left"/>
   <xacro:leg_gazebo_v0 prefix="right"/>
-  <gazebo>
+  <!-- <gazebo>
     <plugin name="left_leg_ClosedLoopPlugin" filename="libpegasus_gazebo_closed_loop_plugin.so">
-      <joint>base_back_joint</joint>
+      <joint>base_back_joint_left</joint>
       <child>side_leg_left</child>
-      <parent>upper_side_leg_left</parent>
-      <position>0.1 0.0 0.0</position>
+      <parent>upper_side_leg_left_opposite</parent>
+      <position>0.0 0.0 0.0</position>
       <rotation>0.00 -0.00 0.00</rotation>
     </plugin>
@@ -60,11 +62,11 @@
   <gazebo>
     <plugin name="right_leg_ClosedLoopPlugin" filename="libpegasus_gazebo_closed_loop_plugin.so">
-      <joint>base_back_joint</joint>
+      <joint>base_back_joint_right</joint>
       <child>side_leg_right</child>
-      <parent>upper_side_leg_right</parent>
-      <position>0.1 0.0 0.0</position>
+      <parent>upper_side_leg_right_opposite</parent>
+      <position>0.0 0.0 0.0</position>
       <rotation>0.00 -0.00 0.00</rotation>
     </plugin>
-  </gazebo>
+  </gazebo> -->
   <!-- Wheel -->
   <xacro:wheel_gazebo_v0 prefix="left"/>

File: echo_bot_description/robots/test.urdf (robot description, URDF)
Before this commit: robot echo_bot, 10 links, 9 joints
Links:
- removed link base_footprint
- added link side_leg_left, mass 0.005; visual box size=0.003 0.003 0.003
- added link side_leg_right, mass 0.005; visual box size=0.003 0.003 0.003
- added link world
- link base_link: mass 1e-05 -> 2.915
- link lower_leg_left: mass 13.25 -> 0.152994; geometry collision mesh filename=package://echo_bot_description/meshes/DAE/lower_leg_left.dae; visual mesh filename=package://echo_bot_description/meshes/STL/lower_leg_left.stl
- link lower_leg_right: mass 13.25 -> 0.152994; geometry collision mesh filename=package://echo_bot_description/meshes/DAE/lower_leg_right.d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; visual mesh filename=package://echo_bot_description/meshes/STL/lower_leg_right.s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
- link upper_leg_left: mass 13.25 -> 0.109
- link upper_leg_right: mass 13.25 -> 0.109
- link upper_side_leg_left: mass 13.25 -> 0.041157
- link upper_side_leg_right: mass 13.25 -> 0.041157
- link wheel_left_link: mass 13.25 -> 0.039831
- link wheel_right_link: mass 13.25 -> 0.039831
Joints:
- added joint side_leg_left_joint: type fixed, parent base_link, child side_leg_left, origin xyz=-0.04 0.0475 0.035 rpy=0 0 0
- added joint side_leg_right_joint: type fixed, parent base_link, child side_leg_right, origin xyz=-0.04 -0.0475 0.035 rpy=0 0 0
- joint base_link_joint: origin xyz=0 0 0.090 -> xyz=0 0 0.20; parent base_footprint -> world
- joint lower_leg_left: mimic joint=upper_leg_left_joint multiplier=-2.186 offset=-0.02025 -> (none)
- joint lower_leg_right: mimic joint=upper_leg_right_joint multiplier=-2.186 offset=-0.02025 -> (none)
- joint upper_side_leg_left: mimic joint=upper_leg_left_joint multiplier=2.123937 offset=0.003625 -> (none)
- joint upper_side_leg_right: mimic joint=upper_leg_right_joint multiplier=2.123937 offset=0.003625 -> (none)
- joint wheel_left_joint: origin xyz=0.1 0.0305 0.0 rpy=-1.57079637 0.0 0.0 -> xyz=0.1 0.0305 0.0 rpy=-1.57079637 0.0 3.14159274

File: echo_bot_description/urdf/base/echo_bot_base.urdf.xacro (robot description, xacro)
@@ -29,6 +29,4 @@
       </inertial>
     </link>
-    <link name="side_leg_left"/>
-    <link name="side_leg_right"/>
     <joint name="base_link_joint" type="fixed">
       <insert_block name="joint_origin"/>
@@ -36,14 +34,4 @@
       <child link="base_link"/>
     </joint>
-    <joint name="side_leg_left_joint" type="fixed">
-      <origin xyz="-0.04 0.0475 0.035" rpy="0 0 0"/>
-      <parent link="base_link"/>
-      <child link="side_leg_left"/>
-    </joint>
-    <joint name="side_leg_right_joint" type="fixed">
-      <origin xyz="-0.04 -0.0475 0.035" rpy="0 0 0"/>
-      <parent link="base_link"/>
-      <child link="side_leg_right"/>
-    </joint>
   </xacro:macro>
 </robot>

File: echo_bot_description/urdf/leg/echo_bot_leg.transmission.xacro (robot description, xacro)
@@ -1,12 +1,22 @@
 <?xml version="1.0"?>
 <robot xmlns:xacro="http://ros.org/wiki/xacro">
-  <xacro:macro name="leg_trans_v0" params="prefix">
-    <transmission name="leg_${prefix}_trans">
+  <xacro:macro name="leg_position_trans_v0" params="joint">
+    <transmission name="${joint}_trans">
       <type>transmission_interface/SimpleTransmission</type>
-      <joint name="upper_leg_${prefix}_joint">
+      <joint name="${joint}">
+        <hardwareInterface>hardware_interface/PositionJointInterface</hardwareInterface>
+      </joint>
+      <actuator name="${joint}_motor">
+        <mechanicalReduction>1</mechanicalReduction>
+      </actuator>
+    </transmission>
+  </xacro:macro>
+  <xacro:macro name="leg_effort_trans_v0" params="joint">
+    <transmission name="${joint}_trans">
+      <type>transmission_interface/SimpleTransmission</type>
+      <joint name="${joint}">
         <hardwareInterface>hardware_interface/EffortJointInterface</hardwareInterface>
       </joint>
-      <actuator name="leg_${prefix}_motor">
-        <hardwareInterface>hardware_interface/EffortJointInterface</hardwareInterface>
+      <actuator name="${joint}_motor">
         <mechanicalReduction>1</mechanicalReduction>
       </actuator>

File: echo_bot_description/urdf/leg/echo_bot_leg.urdf.xacro (robot description, xacro)
@@ -81,6 +81,7 @@
       <child link="upper_leg_${prefix}" />
       <axis xyz="0 1 0"/>
-      <limit lower="0.0" upper="${-M_PI*30/180}" effort="0" velocity="0"/>
+      <limit lower="0.0" upper="${-M_PI*30/180}" effort="1.0" velocity="10.0"/>
     </joint>
+    <xacro:leg_position_trans_v0 joint="upper_leg_${prefix}_joint"/>
     <joint name="lower_leg_${prefix}" type="revolute">
       <origin xyz="0.1 0.0 0.0" rpy="0.0 ${-M_PI*144.47/180} 0.0" />
@@ -88,7 +89,8 @@
       <child link="lower_leg_${prefix}" />
       <axis xyz="0 1 0"/>
-      <limit lower="0.0" upper="${M_PI*66.73/180}" effort="0" velocity="0"/>
-      <mimic joint="upper_leg_${prefix}_joint" multiplier="-2.186" offset="-0.02025"/>
+      <limit lower="0.0" upper="${M_PI*66.73/180}" effort="1.0" velocity="10.0"/>
+      <!-- <mimic joint="upper_leg_${prefix}_joint" multiplier="-2.186" offset="-0.02025"/> -->
     </joint>
+    <xacro:leg_position_trans_v0 joint="lower_leg_${prefix}"/>
     <joint name="upper_side_leg_${prefix}" type="revolute">
       <origin xyz="-0.025 0.0 0.0" rpy="0.0 ${-M_PI*54.22/180} 0.0" />
@@ -96,7 +98,8 @@
       <child link="upper_side_leg_${prefix}" />
       <axis xyz="0 1 0"/>
-      <limit lower="0.0" upper="${-M_PI*64.73/180}" effort="0" velocity="0"/>
-      <mimic joint="upper_leg_${prefix}_joint" multiplier="2.123937" offset="0.003625"/>
+      <limit lower="0.0" upper="${-M_PI*64.73/180}" effort="1.0" velocity="10.0"/>
+      <!-- <mimic joint="upper_leg_${prefix}_joint" multiplier="2.123937" offset="0.003625"/> -->
     </joint>
+    <xacro:leg_position_trans_v0 joint="upper_side_leg_${prefix}"/>
   </xacro:macro>
 </robot>

Commit message: test pegasus (not work)

File: echo_bot_description/robots/echo_bot.urdf.xacro (robot description, xacro)
@@ -6,12 +6,12 @@
   <xacro:include filename="$(find echo_bot_description)/urdf/wheel/echo_bot_wheel.urdf.xacro"/>
   <!-- == echo_bot base == -->
-  <link name="base_footprint"/>
+  <!-- <link name="base_footprint"/>
   <xacro:base_v0 parent="base_footprint">
   <origin xyz="0 0 0.090"/>
-  </xacro:base_v0>
-  <!-- <link name="world"/>
+  </xacro:base_v0> -->
+  <link name="world"/>
   <xacro:base_v0 parent="world">
   <origin xyz="0 0 0.20"/>
-  </xacro:base_v0> -->
+  </xacro:base_v0>
   <!-- == left_leg == -->
   <xacro:leg_v0 parent="base_link" prefix="left">
@@ -51,10 +51,10 @@
   <xacro:leg_gazebo_v0 prefix="left"/>
   <xacro:leg_gazebo_v0 prefix="right"/>
-  <!-- <gazebo>
+  <gazebo>
     <plugin name="left_leg_ClosedLoopPlugin" filename="libpegasus_gazebo_closed_loop_plugin.so">
       <joint>base_back_joint_left</joint>
       <child>side_leg_left</child>
-      <parent>upper_side_leg_left_opposite</parent>
-      <position>0.0 0.0 0.0</position>
+      <parent>upper_side_leg_left</parent>
+      <position>0.1 0.0 0.0</position>
       <rotation>0.00 -0.00 0.00</rotation>
     </plugin>
@@ -64,9 +64,9 @@
       <joint>base_back_joint_right</joint>
       <child>side_leg_right</child>
-      <parent>upper_side_leg_right_opposite</parent>
-      <position>0.0 0.0 0.0</position>
+      <parent>upper_side_leg_right</parent>
+      <position>0.1 0.0 0.0</position>
       <rotation>0.00 -0.00 0.00</rotation>
     </plugin>
-  </gazebo> -->
+  </gazebo>
   <!-- Wheel -->
   <xacro:wheel_gazebo_v0 prefix="left"/>

File: echo_bot_description/urdf/leg/echo_bot_leg.urdf.xacro (robot description, xacro)
@@ -76,30 +76,24 @@
     </link>
     <!-- Joint -->
-    <joint name="upper_leg_${prefix}_joint" type="revolute">
+    <joint name="upper_leg_${prefix}_joint" type="continuous">
       <insert_block name="joint_origin"/>
       <parent link="${parent}" />
       <child link="upper_leg_${prefix}" />
       <axis xyz="0 1 0"/>
-      <limit lower="0.0" upper="${-M_PI*30/180}" effort="30" velocity="${M_PI}"/>
+      <!-- <limit lower="0.0" upper="${-M_PI*30/180}" effort="30" velocity="${M_PI}"/> -->
     </joint>
-    <xacro:leg_position_trans_v0 joint="upper_leg_${prefix}_joint"/>
-    <joint name="lower_leg_${prefix}" type="revolute">
+    <!-- <xacro:leg_position_trans_v0 joint="upper_leg_${prefix}_joint"/> -->
+    <joint name="lower_leg_${prefix}" type="continuous">
       <origin xyz="0.1 0.0 0.0" rpy="0.0 ${-M_PI*144.47/180} 0.0" />
       <parent link="upper_leg_${prefix}" />
       <child link="lower_leg_${prefix}" />
       <axis xyz="0 1 0"/>
-      <limit lower="0.0" upper="${M_PI*66.73/180}" effort="30" velocity="${M_PI}"/>
-      <!-- <mimic joint="upper_leg_${prefix}_joint" multiplier="-2.186" offset="-0.02025"/> -->
     </joint>
-    <xacro:leg_position_trans_v0 joint="lower_leg_${prefix}"/>
-    <joint name="upper_side_leg_${prefix}" type="revolute">
+    <joint name="upper_side_leg_${prefix}" type="continuous">
       <origin xyz="-0.025 0.0 0.0" rpy="0.0 ${-M_PI*54.22/180} 0.0" />
       <parent link="lower_leg_${prefix}" />
       <child link="upper_side_leg_${prefix}" />
       <axis xyz="0 1 0"/>
-      <limit lower="0.0" upper="${-M_PI*64.73/180}" effort="30" velocity="${M_PI}"/>
-      <!-- <mimic joint="upper_leg_${prefix}_joint" multiplier="2.123937" offset="0.003625"/> -->
     </joint>
-    <xacro:leg_position_trans_v0 joint="upper_side_leg_${prefix}"/>
   </xacro:macro>
 </robot>

Commit message: rename & fix link_relation

File: echo_bot_description/robots/echo_bot.urdf.xacro (robot description, xacro)
@@ -2,22 +2,28 @@
 <robot name="echo_bot" xmlns:xacro="http://ros.org/wiki/xacro">
   <xacro:include filename="$(find echo_bot_description)/urdf/common.xacro"/>
-  <xacro:include filename="$(find echo_bot_description)/urdf/base/echo_bot_base.urdf.xacro"/>
+  <xacro:include filename="$(find echo_bot_description)/urdf/torso/echo_bot_torso.urdf.xacro"/>
   <xacro:include filename="$(find echo_bot_description)/urdf/leg/echo_bot_leg.urdf.xacro"/>
   <xacro:include filename="$(find echo_bot_description)/urdf/wheel/echo_bot_wheel.urdf.xacro"/>
   <!-- == echo_bot base == -->
-  <link name="base_footprint"/>
-  <xacro:base_v0 parent="base_footprint">
-  <origin xyz="0 0 0.090"/>
-  </xacro:base_v0>
+  <link name="base_link"/>
+  <xacro:torso_v0 parent="base_link">
+    <origin xyz="0 0 0.090"/>
+  </xacro:torso_v0>
   <!-- <link name="world"/>
-  <xacro:base_v0 parent="world">
+  <xacro:torso_v0 parent="world">
   <origin xyz="0 0 0.20"/>
-  </xacro:base_v0> -->
+  </xacro:torso_v0> -->
+  <!-- <link name="base_footprint"/>
+  <joint name="base_link_to_base_footprint_joint" type="fixed">
+    <origin xyz="0 0 0.090"/>
+    <parent link="base_link"/>
+    <child link="base_footprint"/>
+  </joint> -->
   <!-- == left_leg == -->
-  <xacro:leg_v0 parent="base_link" prefix="left">
+  <xacro:leg_v0 parent="torso_link" prefix="left">
     <origin xyz="0.0 0.0475 0.0" rpy="0.0 ${M_PI*160/180} 0.0"/>
   </xacro:leg_v0>
   <!-- == right_leg == -->
-  <xacro:leg_v0 parent="base_link" prefix="right">
+  <xacro:leg_v0 parent="torso_link" prefix="right">
     <origin xyz="0.0 -0.0475 0.0" rpy="0.0 ${M_PI*160/180} 0.0"/>
   </xacro:leg_v0>
@@ -47,26 +53,8 @@
   </plugin>
   <!-- Base -->
-  <xacro:base_gazebo_v0/>
+  <xacro:torso_gazebo_v0/>
   <!-- leg -->
   <xacro:leg_gazebo_v0 prefix="left"/>
   <xacro:leg_gazebo_v0 prefix="right"/>
-  <!-- <gazebo>
-    <plugin name="left_leg_ClosedLoopPlugin" filename="libpegasus_gazebo_closed_loop_plugin.so">
-      <joint>base_back_joint_left</joint>
-      <child>side_leg_left</child>
-      <parent>upper_side_leg_left_opposite</parent>
-      <position>0.0 0.0 0.0</position>
-      <rotation>0.00 -0.00 0.00</rotation>
-    </plugin>
-  </gazebo>
-  <gazebo>
-    <plugin name="right_leg_ClosedLoopPlugin" filename="libpegasus_gazebo_closed_loop_plugin.so">
-      <joint>base_back_joint_right</joint>
-      <child>side_leg_right</child>
-      <parent>upper_side_leg_right_opposite</parent>
-      <position>0.0 0.0 0.0</position>
-      <rotation>0.00 -0.00 0.00</rotation>
-    </plugin>
-  </gazebo> -->
   <!-- Wheel -->
   <xacro:wheel_gazebo_v0 prefix="left"/>

File: echo_bot_description/robots/test.urdf (robot description, URDF)
Before this commit: robot echo_bot, 10 links, 9 joints
Links:
- removed link base_footprint
- added link torso_link, mass 2.915; collision mesh filename=package://echo_bot_description/meshes/STL/torso.stl; visual mesh filename=package://echo_bot_description/meshes/DAE/torso.dae
- link base_link: mass 2.915 -> None; geometry 
- link wheel_left_link: mass None -> 0.039831; geometry collision cylinder length=0.012 radius=0.029; visual mesh filename=package://echo_bot_description/meshes/DAE/tyre.dae
- link wheel_right_link: mass None -> 0.039831; geometry collision cylinder length=0.012 radius=0.029; visual mesh filename=package://echo_bot_description/meshes/DAE/tyre.dae
Joints:
- joint base_link_joint: child base_link -> torso_link; parent base_footprint -> base_link
- joint upper_leg_left_joint: parent base_link -> torso_link
- joint upper_leg_right_joint: parent base_link -> torso_link

File: echo_bot_description/urdf/torso/echo_bot_torso.gazebo.xacro (robot description, xacro)
@@ -1,6 +1,6 @@
 <?xml version="1.0"?>
 <robot xmlns:xacro="http://ros.org/wiki/xacro">
-  <xacro:macro name="base_gazebo_v0">
-    <gazebo reference="base_link">
+  <xacro:macro name="torso_gazebo_v0">
+    <gazebo reference="torso_link">
       <selfCollide>true</selfCollide>
       <mu1 value="0.05" />

File: echo_bot_description/urdf/torso/echo_bot_torso.urdf.xacro (robot description, xacro)
@@ -2,15 +2,15 @@
 <robot xmlns:xacro="http://ros.org/wiki/xacro">
   <!-- == Material == -->
-  <material name="base_color">
+  <material name="torso_color">
     <color rgba="0.3 0.3 0.3 1"/>
   </material>
-  <xacro:include filename="$(find echo_bot_description)/urdf/base/echo_bot_base.gazebo.xacro"/>
-  <xacro:macro name="base_v0" params="parent *joint_origin">
-    <link name="base_link">
+  <xacro:include filename="$(find echo_bot_description)/urdf/torso/echo_bot_torso.gazebo.xacro"/>
+  <xacro:macro name="torso_v0" params="parent *joint_origin">
+    <link name="torso_link">
       <visual>
         <origin rpy="0 0 0"/>
-        <material name="base_color"/>
+        <material name="torso_color"/>
         <geometry>
-          <mesh filename="package://echo_bot_description/meshes/DAE/body.dae"/>
+          <mesh filename="package://echo_bot_description/meshes/DAE/torso.dae"/>
         </geometry>
       </visual>
@@ -18,5 +18,5 @@
         <origin rpy="0 0 0"/>
         <geometry>
-          <mesh filename="package://echo_bot_description/meshes/STL/body.stl"/>
+          <mesh filename="package://echo_bot_description/meshes/STL/torso.stl"/>
         </geometry>
       </collision>
@@ -32,5 +32,5 @@
       <insert_block name="joint_origin"/>
       <parent link="${parent}"/>
-      <child link="base_link"/>
+      <child link="torso_link"/>
     </joint>
   </xacro:macro>

File: echo_bot_description/urdf/wheel/echo_bot_wheel.gazebo.xacro (robot description, xacro)
@@ -4,10 +4,6 @@
     <gazebo reference="wheel_${prefix}_link">
       <selfCollide>true</selfCollide>
-      <!-- <mu1 value="0.8" />
-      <mu2 value="0.8" /> -->
-      <mu1 value="2.5" />
-      <mu2 value="2.5" />
-      <kp value="50000" />
-      <kd value="10" />
+      <mu1 value="0.8" />
+      <mu2 value="0.8" />
     </gazebo>
   </xacro:macro>

Commit message: cmd_vel動いた

File: echo_bot_description/robots/echo_bot.urdf.xacro (robot description, xacro)
@@ -30,5 +30,5 @@
   <!-- == left_wheel == -->
   <xacro:wheel_v0 prefix="left" parent="lower_leg_left">
-    <origin xyz="0.1 0.0305 0.0" rpy="${-M_PI/2} 0.0 ${M_PI}"/>
+    <origin xyz="0.1 0.0305 0.0" rpy="${-M_PI/2} 0.0 0.0"/>
     <axis xyz="0 0 1"/>
   </xacro:wheel_v0>

File: echo_bot_description/urdf/wheel/echo_bot_wheel.gazebo.xacro (robot description, xacro)
@@ -4,6 +4,6 @@
     <gazebo reference="wheel_${prefix}_link">
       <selfCollide>true</selfCollide>
-      <mu1 value="0.8" />
-      <mu2 value="0.8" />
+      <mu1 value="1.5" />
+      <mu2 value="1.5" />
     </gazebo>
   </xacro:macro>

Commit message: worldに貼り付け

File: echo_bot_description/robots/echo_bot.urdf.xacro (robot description, xacro)
@@ -6,12 +6,12 @@
   <xacro:include filename="$(find echo_bot_description)/urdf/wheel/echo_bot_wheel.urdf.xacro"/>
   <!-- == echo_bot base == -->
-  <link name="base_link"/>
+  <!-- <link name="base_link"/>
   <xacro:torso_v0 parent="base_link">
     <origin xyz="0 0 0.090"/>
-  </xacro:torso_v0>
-  <!-- <link name="world"/>
+  </xacro:torso_v0> -->
+  <link name="world"/>
   <xacro:torso_v0 parent="world">
   <origin xyz="0 0 0.20"/>
-  </xacro:torso_v0> -->
+  </xacro:torso_v0>
   <!-- <link name="base_footprint"/>
   <joint name="base_link_to_base_footprint_joint" type="fixed">
